File: Electrical/KiCad_templates/Expansion_Card_Retrofit/Expansion_Card_rs-probe.kicad_sch (KiCad schematic)
At the start: 94 parts, among them J10 Conn_01x01, J11 Conn_01x01, J5 tag-connect-swd, J6 Conn_01x01, J7 Conn_01x01, J8 Conn_01x01, J9 Conn_01x01, P1 USB_C_Plug_USB2.0, Q1 NTZD3155C or CMLDM3757-TR-PBF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, SW1 EVQ-P2002W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

Commit message: VCP and 3d models
Parts:
- added J1: Conn_01x04, Connector_PinHeader_1.00mm:PinHeader_1x04_P1.00mm_Vertical_SMD_Pin1Left, symbol Connector_Generic_MountingPin:Conn_01x04_MountingPin
- added U1, U2: 74LVC1T45GM,115, Package_TO_SOT_SMD:SOT-886, symbol rs-probe:74LVC1T45
- SW1: value EVQ-P2002W -> B3U-1000P; footprint Button_Switch_SMD:SW_SPST_EVQP2 -> Button_Switch_SMD:SW_SPST_B3U-1000P
Connections:
- net +3.3V: now also U1.1 (VCCA), U2.1 (VCCA)
- net GND: now also J1.1 (Pin_1), J1.MP (MountPin), U1.2 (GND), U2.2 (GND)
- net TRANS_VCC: now also U1.6 (VCCB), U2.6 (VCCB)
- net T_VCC: now also J1.2 (Pin_2)
- net T_VCP_RX: now also U4.16 (1B), J1.4 (Pin_4)
- net T_VCP_TX: now also U4.15 (2B), J1.3 (Pin_3)
- net VCP_TX: now reaches U6.31 (GPIO20)
- net VCP_TX: now also U2.3 (A)
- net VCP_RX: now reaches U6.32 (GPIO21)
- net VCP_RX: now also U1.3 (A)
- net DIR_VCP_TX: now reaches U6.36 (GPIO24)
- net DIR_VCP_TX: now also U2.5 (DIR)
- net DIR_VCP_RX: now reaches U6.37 (GPIO25)
- net DIR_VCP_RX: now also U1.5 (DIR)
- net at U4.1 (1A): now also U1.4 (B)
- net at U4.2 (2A): now also U2.4 (B)
- no-connect marks 18 -> 10
