File: Electrical/KiCad_templates/Expansion_Card_Retrofit/Expansion_Card_rs-probe.kicad_pcb (KiCad board)
At the start: 2 copper layers, 24 x 27.3 mm, 86 parts, among them J5 tag-connect-swd, P1 USB_C_Plug_USB2.0, Q1 NTZD3155C or CMLDM3757-TR-PBF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, SW1 EVQ-P2002W, U10 74LVC1T45GM,115, U11 74LVC1T45GM,115, U12 NCP133AMXADJTCG, U13 NCP133AMXADJTCG, U14 NCP133AMXADJTCG, U3 W25Q8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

Commit message: VCP and 3d models
Parts:
- added J1: Conn_01x04, Connector_PinHeader_1.00mm:PinHeader_1x04_P1.00mm_Vertical_SMD_Pin1Left, F.Cu at (146.6, 152.5)
- added U1: 74LVC1T45GM,115, Package_TO_SOT_SMD:SOT-886, F.Cu at (148.9, 142.8)
- added U2: 74LVC1T45GM,115, Package_TO_SOT_SMD:SOT-886, F.Cu at (150.7, 142.8)
- SW1: value EVQ-P2002W -> B3U-1000P; footprint Button_Switch_SMD:SW_SPST_EVQP2 -> Button_Switch_SMD:SW_SPST_B3U-1000P
- moved R23 11.6 mm to (134.8, 149.8), turned to 180 degrees
- moved R24 8.80 mm to (136.8, 149.8), turned to 0 degrees
- moved R19 8.43 mm to (141.6, 153.8), turned to 180 degrees
- moved Q1 6.93 mm to (141.6, 152.4), turned to 0 degrees
- moved R10 6.11 mm to (138.8, 149.8), turned to 180 degrees
- moved R20 5.76 mm to (141.6, 151.0), turned to 180 degrees
- moved D2 5.64 mm to (148.0, 145.2), turned to 180 degrees
- moved C17 5.32 mm to (148.3, 146.5), turned to 90 degrees
- moved U5 3.80 mm to (136.2, 154.4)
- moved C16 2.66 mm to (148.3, 148.5), turned to -90 degrees
- moved SW1 2.10 mm to (130.9, 152.6), turned to 0 degrees
- moved R11 2.10 mm to (132.3, 149.2)
- moved R22 2.10 mm to (133.1, 149.2)
- moved R9 2.10 mm to (131.5, 149.2)
- moved J5 1.63 mm to (150.0, 137.4)
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Connections:
- U4 pad 1: unconnected-(U4-1A-Pad1) -> Net-(U1-B)
- U4 pad 15: unconnected-(U4-2B-Pad15) -> /T_VCP_TX
- U4 pad 16: unconnected-(U4-1B-Pad16) -> /T_VCP_RX
- U4 pad 2: unconnected-(U4-2A-Pad2) -> Net-(U2-B)
- U6 pad 31: unconnected-(U6-GPIO20-Pad31) -> /VCP_TX
- U6 pad 32: unconnected-(U6-GPIO21-Pad32) -> /VCP_RX
- U6 pad 36: unconnected-(U6-GPIO24-Pad36) -> /DIR_VCP_TX
- U6 pad 37: unconnected-(U6-GPIO25-Pad37) -> /DIR_VCP_RX
Routing:
- net /PROTECTED_5V: track 2.14 -> 18.9 mm, vias 0 -> 2
- net Net-(U2-B): track 0.00 -> 15.5 mm, vias 0 -> 2
- net Net-(U1-B): track 0.00 -> 15.0 mm, vias 0 -> 2
- net /5V_KEY_EN: track 35.1 -> 45.9 mm, vias 2 -> 4
- net /TRANS_VCC: track 37.5 -> 48.2 mm, vias 8 -> 10
- net /DIR_VCP_TX: track 0.00 -> 10.3 mm, vias 0 -> 2
- net /T_VCP_RX: track 0.00 -> 9.31 mm
- net /DIR_VCP_RX: track 0.00 -> 9.23 mm, vias 0 -> 2
- net +3.3V: track 105.2 -> 114.2 mm, vias 10 -> 12
- net /VCP_TX: track 0.00 -> 8.90 mm
- net /T_VCP_TX: track 0.00 -> 8.72 mm
- net /5V_KEY: track 14.6 -> 7.65 mm
- net /T_SWO_TDO: track 12.1 -> 5.29 mm, vias 2 -> 0
- net /VCP_RX: track 0.00 -> 6.42 mm
- net /T_SWDCLK_JCLK: track 13.8 -> 7.51 mm, vias 2 -> 0
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
Commit message: v0 ordered
Parts:
- added T1: Tab, kikit:Tab, F.Cu at (3.15, 1.15)
- added T2: Tab, kikit:Tab, F.Cu at (3.15, 4.45)
- U6: footprint qfn:RP2040-QFN-56 -> Package_DFN_QFN:QFN-56-1EP_7x7mm_P0.4mm_EP3.2x3.2mm_ThermalVias
- moved X1 0.15 mm to (138.5, 144.9)
Routing:
- net +3.3V: track 114.2 -> 81.3 mm
- net /T_VCC: track 26.2 -> 42.0 mm
- added copper zone on F.Cu, net +3.3V
